File: PCB/SnakeBoy/_autosave-SnakeBoy.kicad_pcb (KiCad board)
At the start: 2 copper layers, 15 parts, among them SW1 SW_Push, SW2 SW_Push, SW3 SW_Push, SW4 SW_Push, SW5 SW_Push, SW6 SW_Push, SW7 SW_DIP_x01, U1 ESP32-S3-DEVKITC-1-N16R8, U2 COM-09032, U3 PAM8304 Module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

Commit message: Finished the Controller and Display schems
Parts:
- moved U2 21.6 mm to (256.5, 147.3), turned to -90 degrees
